File: Camera/CameraSlave_KiCad/ThermalCamera.kicad_sch (KiCad schematic)
At the start: 40 parts, among them J1 I2C, J10 Cam 2, J11 XT60 Header, J12 XT60 Header, J13 XT60 Header, J14 ICSP, J2 XT60 Header, J3 Cam 1, J4 Conn_Coaxial, J5 Fan, J6 I2C, J7 RGB, J8 Cam 3, J9 Cam 4, U2 TLV1117-50, U3 4052, U4 LMH6574, U5 LT1171

Commit message: adding finished board schematic as well as PCB design
Parts:
- removed J4: Conn_Coaxial, symbol Connector:Conn_Coaxial
- added C10, C2, C4: .1uF, 1FootPrintLibrary:0805, symbol Device:C
- added C11: 10pF, 1FootPrintLibrary:0805, symbol Device:C_US
- added C3: 1uF, 1FootPrintLibrary:0805, symbol Device:C_US
- added C7: 1uf, 1FootPrintLibrary:0805, symbol Device:C
- added D3: 1N4148, 1FootPrintLibrary:DIODE_0805, symbol Device:D_Filled
- added J16: TX PWR, 1FootPrintLibrary:Header_1_x_2, symbol 1_Library:2Pin_Header
- added J6: XT60 Header, 1FootPrintLibrary:XT-60 Power Male (Load Side), symbol 1_Library:XT60
- added J8: TX Female, 1FootPrintLibrary:Header_1_x_3, symbol 1_Library:3Pin_Header
- added R2: 470 1W, Resistor_THT:R_Axial_DIN0309_L9.0mm_D3.2mm_P12.70mm_Horizontal, symbol Device:R_US
- added R6: 10k, 1FootPrintLibrary:0805, symbol Device:R_US
- C1: footprint (none) -> Capacitor_THT:C_Radial_D5.0mm_H11.0mm_P2.00mm
- C5: renamed from C3; footprint (none) -> 1FootPrintLibrary:0805
- C6: renamed from C2; footprint (none) -> Capacitor_THT:C_Radial_D5.0mm_H11.0mm_P2.00mm
- C8: renamed from C4; footprint (none) -> 1FootPrintLibrary:0805
- C9: renamed from C5; value 680uF -> 330uF; footprint (none) -> Capacitor_THT:C_Radial_D8.0mm_H11.5mm_P3.50mm
- D1: renamed from D2; footprint (none) -> 1FootPrintLibrary:DIODE_0805
- D2: renamed from D1; footprint (none) -> 1FootPrintLibrary:DIODE_0805
- D4: renamed from D3; value 1N4001 -> 1N914; footprint (none) -> 1FootPrintLibrary:DIODE_0805
- D5: renamed from D4; value 1N4001 -> 1N914; footprint (none) -> 1FootPrintLibrary:DIODE_0805
- J1: footprint (none) -> 1FootPrintLibrary:Header_1_x_4
- J10: footprint (none) -> 1FootPrintLibrary:Header_1_x_7
- J11: renamed from J8; footprint (none) -> 1FootPrintLibrary:Header_1_x_7
- J12: renamed from J9; footprint (none) -> 1FootPrintLibrary:Header_1_x_7
- J13: renamed from J7; footprint (none) -> 1FootPrintLibrary:Header_1_x_4
- J14: renamed from J5; footprint (none) -> 1FootPrintLibrary:Header_1_x_4
- J15: renamed from J6; footprint (none) -> 1FootPrintLibrary:Header_1_x_4
- J2: footprint (none) -> 1FootPrintLibrary:XT-60 Power Male (Load Side)
- J3: renamed from J11; footprint (none) -> 1FootPrintLibrary:XT-60 Power Male (Load Side)
- J4: renamed from J12; footprint (none) -> 1FootPrintLibrary:XT-60 Power Male (Load Side)
- J5: renamed from J13; footprint (none) -> 1FootPrintLibrary:XT-60 Power Male (Load Side)
- J7: renamed from J14; footprint (none) -> 1FootPrintLibrary:Header_1_x_6
- J9: renamed from J3; footprint (none) -> 1FootPrintLibrary:Header_1_x_7
- L1: renamed from L2; footprint (none) -> 1FootPrintLibrary:78404064680
- L2: renamed from L1; footprint (none) -> 1FootPrintLibrary:0805
- R1: renamed from R6; value 1.5k -> 5.1k; footprint (none) -> 1FootPrintLibrary:0805
- R10: renamed from R5; footprint (none) -> 1FootPrintLibrary:0805
- R11: renamed from R2; footprint (none) -> 1FootPrintLibrary:0805
- R12: renamed from R3; footprint (none) -> 1FootPrintLibrary:0805
- R3: renamed from R1; footprint (none) -> 1FootPrintLibrary:0805
- R4: renamed from R7; value 1.24k -> 1.2k; footprint (none) -> 1FootPrintLibrary:0805
- R5: renamed from R8; value 10.7k -> 3.9k; footprint (none) -> 1FootPrintLibrary:0805
- R7: renamed from R9; footprint (none) -> 1FootPrintLibrary:0805
- R8: renamed from R10; value 100 -> 100 1W; footprint (none) -> Resistor_THT:R_Axial_DIN0309_L9.0mm_D3.2mm_P12.70mm_Horizontal
- R9: renamed from R4; footprint (none) -> 1FootPrintLibrary:0805
- U1: renamed from U2; footprint (none) -> 1FootPrintLibrary:TLV1117-50
- U2: renamed from U5; footprint (none) -> 1FootPrintLibrary:LT1172
- U3: renamed from U1; footprint (none) -> 1FootPrintLibrary:PIC16F883
- U4: renamed from U3; footprint (none) -> 1FootPrintLibrary:CD4052BPWR
- U5: renamed from U4; footprint (none) -> 1FootPrintLibrary:LMH6574
Connections:
- net GND: now also C10.1, C2.2, C4.2, C7.2, J16.2, J6.2 (-), J8.1
- net +5V: now reaches C6.1, D2.2 (A), U1.2 (VO)
- net +5V: now also J1.1, J15.1, J7.2, U3.20 (VDD), U4.16 (VDD), U5.14 (V+), C4.1, R6.1
- net +13V: now reaches C1.1, J2.1 (+), U1.3 (VI)
- net +13V: now also J10.3 (PWR), J11.3 (PWR), J12.3 (PWR), J13.1, J14.2, J3.1 (+), J4.1 (+), J5.1 (+), J9.3 (PWR), U2.7 (VSW), C2.1, J16.1, J6.1 (+), R2.2
- net at D1.1 (K), U2.5 (VIN): now also C3.1, R2.1; no longer U2.7 (VSW)
- net at C5.2, C8.2, D5.1 (K)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: now also C3.2
- net at L2.1, R9.1, U5.13 (OUT): now also C11.1
- net at L2.2: now also J8.3
- net at J7.1, U3.1 (RE3/~{MCLR}/Vpp): now also D3.1 (K)
- net -5V: now reaches C9.2, D5.2 (A), R8.2
- net -5V: now also U5.6 (V-), C10.2
- net at R10.1, R9.2, U5.12 (FB): now also C11.2
- new net: C7.1, D3.2 (A), R6.2
- no-connect marks 21 -> 22
Other:
- note added: "*Note a 13V Supply has to be connected to this board for it to function*"
- note added: "13V in"
- moved on the sheet: D1, L2, R8

Commit message: Adding functionality to the zoom for the sony cameras to stop the zoom if it has started, also fixed the homing of the camera
Parts:
- added R10, R9: 330, 1FootPrintLibrary:0805, symbol Device:R_US
- added TP1: 13V, 1FootPrintLibrary:Header_1_x_1, symbol Connector:TestPoint
- added TP10: Video Out, 1FootPrintLibrary:Header_1_x_1, symbol Connector:TestPoint
- added TP11, TP12, TP13: GND, 1FootPrintLibrary:Header_1_x_1, symbol Connector:TestPoint
- added TP2: SCL, 1FootPrintLibrary:Header_1_x_1, symbol Connector:TestPoint
- added TP3: SDA, 1FootPrintLibrary:Header_1_x_1, symbol Connector:TestPoint
- added TP4: 5V, 1FootPrintLibrary:Header_1_x_1, symbol Connector:TestPoint
- added TP5: TX Cam, 1FootPrintLibrary:Header_1_x_1, symbol Connector:TestPoint
- added TP6: RX Cam, 1FootPrintLibrary:Header_1_x_1, symbol Connector:TestPoint
- added TP7: -5V, 1FootPrintLibrary:Header_1_x_1, symbol Connector:TestPoint
- added TP8: RB0, 1FootPrintLibrary:Header_1_x_1, symbol Connector:TestPoint
- added TP9: RB1, 1FootPrintLibrary:Header_1_x_1, symbol Connector:TestPoint
- renumbered R9 to R11, R10 to R12, R11 to R13, R12 to R14
Connections:
- net +13V: now also TP1.1
- net +5V: now also TP4.1
- net -5V: now also TP7.1
- net GND: now also R10.2, R9.2, TP11.1, TP12.1, TP13.1
- net RB0: now also R9.1, TP8.1
- net RB1: now also R10.1, TP9.1
- net SCL: now also TP2.1
- net SDA: now also TP3.1
- net at J8.3, L2.2: now also TP10.1
- net at U3.17 (RC6/TX/CK), U4.13 (X): now also TP5.1
- net at U3.18 (RC7/RX/DT), U4.3 (Y): now also TP6.1
